File: pcb/RPi_GPIO.sch (KiCad schematic (older format))
At the start: 27 parts, among them J1 RPi_GPIO, P1 Flow Meter, P2 Extra, P3 1 Wire, P4 Display, P5 Laser Controller, Q1 BSS138, Q2 PN2222A, Q3 BSS138, Q4 BSS138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

Commit message: Schematic updates
Don't use a relay, use a level shifter so the pin can be used as either
an input or an output.
Parts:
- removed D1: DIODE, Diodes_SMD:SMA_Handsoldering, symbol DIODE
- removed Q2: PN2222A, TO_SOT_Packages_SMD:SOT-23, symbol PN2222A
- removed RL1: G5Q-14, Relays:Relay_SPDS_OMRON-G5Q, symbol G5Q-14
- added Q2: BSS138, TO_SOT_Packages_SMD:SOT-23, symbol BSS138
- added R3: 10k, Resistors_SMD:R_1206_HandSoldering, symbol R
- P2: symbol CONN_01X05 -> CONN_01X04
- R4: value 1k -> 10k
Connections:
- net LP2 is gone; now on net EP1: P2.3 (P3)
- net +3V3: now also Q2.1 (G), R3.2
- net +5V: now also P2.4 (P4), R4.1; no longer P2.5 (P5)
- net EP1: no longer P2.4 (P4)
- net LIGHTS: now also Q2.2 (S), R3.1; no longer R4.2
- net LP1: now also R4.2, Q2.3 (D)
- net FLOW_INPUT: now reaches P1.2 (P2), Q3.3 (D), R6.2
- no-connect marks 28 -> 27
Other:
- moved on the sheet: P1
Changed lines of the file:
@@
 LIBS:power
 LIBS:device
-LIBS:transistors
 LIBS:conn
 LIBS:linear
@@
 LIBS:Xicor
 LIBS:Zilog
+LIBS:Transistors
 LIBS:RPi_Hat-cache
 EELAYER 25 0
@@
 L CONN_01X03 P1
 U 1 1 56EB7785
-P 4650 4450
-F 0 "P1" H 4650 4650 50  0000 C CNN
-F 1 "Flow Meter" V 4750 4450 50  0000 C CNN
-F 2 "Terminal_Blocks:TerminalBlock_Pheonix_MPT-2.54mm_3pol" H 4650 4450 50  0001 C CNN
-F 3 "" H 4650 4450 50  0000 C CNN
-	1    4650 4450
-	0    1    1    0
+P 6750 1750
+F 0 "P1" H 6750 1950 50  0000 C CNN
+F 1 "Flow Meter" V 6850 1750 50  0000 C CNN
+F 2 "Terminal_Blocks:TerminalBlock_Pheonix_MPT-2.54mm_3pol" H 6750 1750 50  0001 C CNN
+F 3 "" H 6750 1750 50  0000 C CNN
+	1    6750 1750
+	0    -1   -1   0
 $EndComp
 Text GLabel 6300 2600 0    60   Input ~ 0
@@
 L GND #PWR014
 U 1 1 56ECCF2D
-P 4900 4250
-F 0 "#PWR014" H 4900 4000 50  0001 C CNN
-F 1 "GND" H 4900 4100 50  0000 C CNN
-F 2 "" H 4900 4250 50  0000 C CNN
-F 3 "" H 4900 4250 50  0000 C CNN
-	1    4900 4250
-	0    -1   -1   0
+P 6650 1950
+F 0 "#PWR014" H 6650 1700 50  0001 C CNN
+F 1 "GND" H 6650 1800 50  0000 C CNN
+F 2 "" H 6650 1950 50  0000 C CNN
+F 3 "" H 6650 1950 50  0000 C CNN
+	1    6650 1950
+	0    1    1    0
 $EndComp
 $Comp
 L +5V #PWR015
 U 1 1 56ECD7DE
-P 4550 4250
-F 0 "#PWR015" H 4550 4100 50  0001 C CNN
-F 1 "+5V" H 4550 4390 50  0000 C CNN
-F 2 "" H 4550 4250 50  0000 C CNN
-F 3 "" H 4550 4250 50  0000 C CNN
-	1    4550 4250
-	0    -1   -1   0
+P 6850 1950
+F 0 "#PWR015" H 6850 1800 50  0001 C CNN
+F 1 "+5V" H 6850 2090 50  0000 C CNN
+F 2 "" H 6850 1950 50  0000 C CNN
+F 3 "" H 6850 1950 50  0000 C CNN
+	1    6850 1950
+	0    1    1    0
 $EndComp
 $Comp
@@
 Text GLabel 9450 1700 2    60   Input ~ 0
 ID_SC
-$Comp
-L R R4
-U 1 1 56FB3E8A
-P 2500 3150
-F 0 "R4" V 2580 3150 50  0000 C CNN
-F 1 "1k" V 2500 3150 50  0000 C CNN
-F 2 "Resistors_SMD:R_1206_HandSoldering" V 2430 3150 50  0001 C CNN
-F 3 "" H 2500 3150 50  0000 C CNN
-	1    2500 3150
-	0    1    1    0
-$EndComp
-Text GLabel 2350 3150 0    60   Input ~ 0
+Text GLabel 4400 2250 0    60   Input ~ 0
 LIGHTS
 Text GLabel 7300 3300 0    60   Input ~ 0
@@
 MC_EXTRA_1
 $Comp
-L CONN_01X05 P2
+L CONN_01X04 P2
 U 1 1 56FBB1F9
 P 5950 1700
@@
 L GND #PWR021
 U 1 1 56FBB492
-P 5750 1900
-F 0 "#PWR021" H 5750 1650 50  0001 C CNN
-F 1 "GND" H 5750 1750 50  0000 C CNN
-F 2 "" H 5750 1900 50  0000 C CNN
-F 3 "" H 5750 1900 50  0000 C CNN
-	1    5750 1900
+P 5800 1900
+F 0 "#PWR021" H 5800 1650 50  0001 C CNN
+F 1 "GND" H 5800 1750 50  0000 C CNN
+F 2 "" H 5800 1900 50  0000 C CNN
+F 3 "" H 5800 1900 50  0000 C CNN
+	1    5800 1900
 	1    0    0    -1
 $EndComp
@@
 L +5V #PWR022
 U 1 1 56FBBB25
-P 6150 1900
-F 0 "#PWR022" H 6150 1750 50  0001 C CNN
-F 1 "+5V" H 6150 2040 50  0000 C CNN
-F 2 "" H 6150 1900 50  0000 C CNN
-F 3 "" H 6150 1900 50  0000 C CNN
-	1    6150 1900
+P 6100 1900
+F 0 "#PWR022" H 6100 1750 50  0001 C CNN
+F 1 "+5V" H 6100 2040 50  0000 C CNN
+F 2 "" H 6100 1900 50  0000 C CNN
+F 3 "" H 6100 1900 50  0000 C CNN
+	1    6100 1900
 	-1   0    0    1
 $EndComp
-Text GLabel 6050 1900 3    60   Input ~ 0
+Text GLabel 6000 1900 3    60   Input ~ 0
 EP1
-Text GLabel 5850 1900 3    60   Input ~ 0
+Text GLabel 5900 1900 3    60   Input ~ 0
 LP1
 $Comp
@@
 $Comp
 L +5V #PWR024
-U 1 1 56FBEB4D
-P 2950 2300
-F 0 "#PWR024" H 2950 2150 50  0001 C CNN
-F 1 "+5V" H 2950 2440 50  0000 C CNN
-F 2 "" H 2950 2300 50  0000 C CNN
-F 3 "" H 2950 2300 50  0000 C CNN
-	1    2950 2300
-	1    0    0    -1
-$EndComp
-$Comp
-L +5V #PWR025
 U 1 1 56FBEBA3
 P 4750 1600
-F 0 "#PWR025" H 4750 1450 50  0001 C CNN
+F 0 "#PWR024" H 4750 1450 50  0001 C CNN
 F 1 "+5V" H 4750 1740 50  0000 C CNN
 F 2 "" H 4750 1600 50  0000 C CNN
@@
 $EndComp
 $Comp
-L GND #PWR026
+L GND #PWR025
 U 1 1 56FC92A9
 P 7600 2100
-F 0 "#PWR026" H 7600 1850 50  0001 C CNN
+F 0 "#PWR025" H 7600 1850 50  0001 C CNN
 F 1 "GND" H 7600 1950 50  0000 C CNN
 F 2 "" H 7600 2100 50  0000 C CNN
@@
 $EndComp
 $Comp
-L +5V #PWR027
+L +5V #PWR026
 U 1 1 56FC943A
 P 7700 2100
-F 0 "#PWR027" H 7700 1950 50  0001 C CNN
+F 0 "#PWR026" H 7700 1950 50  0001 C CNN
 F 1 "+5V" H 7700 2240 50  0000 C CNN
 F 2 "" H 7700 2100 50  0000 C CNN
@@
 NoConn ~ 7300 2700
 NoConn ~ 7300 3000
-$Comp
-L G5Q-14 RL1
-U 1 1 570055E9
-P 3150 2650
-F 0 "RL1" H 3600 2800 50  0000 L CNN
-F 1 "G5Q-14" H 3600 2700 50  0000 L CNN
-F 2 "Relays:Relay_SPDS_OMRON-G5Q" H 3150 2650 50  0001 C CNN
-F 3 "" H 3150 2650 50  0000 C CNN
-	1    3150 2650
-	1    0    0    -1
-$EndComp
-$Comp
-L PN2222A Q2
-U 1 1 57006D52
-P 2850 3150
-F 0 "Q2" H 3050 3225 50  0000 L CNN
-F 1 "PN2222A" H 3050 3150 50  0000 L CNN
-F 2 "TO_SOT_Packages_SMD:SOT-23" H 3050 3075 50  0001 L CIN
-F 3 "" H 2850 3150 50  0000 L CNN
-	1    2850 3150
-	1    0    0    -1
-$EndComp
-$Comp
-L GND #PWR028
-U 1 1 57007675
-P 2950 3350
-F 0 "#PWR028" H 2950 3100 50  0001 C CNN
-F 1 "GND" H 2950 3200 50  0000 C CNN
-F 2 "" H 2950 3350 50  0000 C CNN
-F 3 "" H 2950 3350 50  0000 C CNN
-	1    2950 3350
-	1    0    0    -1
-$EndComp
-Text GLabel 5950 1900 3    60   Input ~ 0
-LP2
-Text GLabel 3350 2950 2    60   Input ~ 0
-LP1
-Text GLabel 3450 2350 2    60   Input ~ 0
-LP2
-$Comp
-L DIODE D1
-U 1 1 57009B19
-P 2550 2650
-F 0 "D1" H 2550 2800 50  0000 C CNN
-F 1 "DIODE" H 2550 2475 50  0000 C CNN
-F 2 "Diodes_SMD:SMA_Handsoldering" H 2550 2650 50  0001 C CNN
-F 3 "" H 2550 2650 50  0000 C CNN
-	1    2550 2650
-	0    1    1    0
-$EndComp
-NoConn ~ 3250 2350
 Wire Wire Line
 	4650 3700 4750 3700
@@
 	4350 1200 4350 1050
 Wire Wire Line
-	2550 2850 2550 2950
-Wire Wire Line
-	2550 2950 2950 2950
-Connection ~ 2950 2350
-Wire Wire Line
-	2550 2450 2550 2350
-Wire Wire Line
-	2550 2350 2950 2350
-Wire Wire Line
-	2950 2350 2950 2300
-Wire Wire Line
-	4750 4250 4900 4250
-Wire Wire Line
-	4650 4100 4650 4250
-Wire Wire Line
 	6300 2850 6650 2850
+$Comp
+L BSS138 Q2
+U 1 1 5703ABB6
+P 4500 2600
+F 0 "Q2" H 4700 2675 50  0000 L CNN
+F 1 "BSS138" H 4700 2600 50  0000 L CNN
+F 2 "TO_SOT_Packages_SMD:SOT-23" H 4700 2525 50  0001 L CIN
+F 3 "" H 4500 2600 50  0000 L CNN
+	1    4500 2600
+	-1   0    0    1
+$EndComp
+$Comp
+L R R4
+U 1 1 5703ABBC
+P 4650 2800
+F 0 "R4" V 4730 2800 50  0000 C CNN
+F 1 "10k" V 4650 2800 50  0000 C CNN
+F 2 "Resistors_SMD:R_1206_HandSoldering" V 4580 2800 50  0001 C CNN
+F 3 "" H 4650 2800 50  0000 C CNN
+	1    4650 2800
+	0    1    1    0
+$EndComp
+$Comp
+L R R3
+U 1 1 5703ABC2
+P 4650 2400
+F 0 "R3" V 4730 2400 50  0000 C CNN
+F 1 "10k" V 4650 2400 50  0000 C CNN
+F 2 "Resistors_SMD:R_1206_HandSoldering" V 4580 2400 50  0001 C CNN
+F 3 "" H 4650 2400 50  0000 C CNN
+	1    4650 2400
+	0    -1   -1   0
+$EndComp
+Text GLabel 4400 2800 3    60   Input ~ 0
+LP1
+$Comp
+L +3.3V #PWR027
+U 1 1 5703ABCA
+P 4800 2400
+F 0 "#PWR027" H 4800 2250 50  0001 C CNN
+F 1 "+3.3V" H 4800 2540 50  0000 C CNN
+F 2 "" H 4800 2400 50  0000 C CNN
+F 3 "" H 4800 2400 50  0000 C CNN
+	1    4800 2400
+	0    1    1    0
+$EndComp
+$Comp
+L +5V #PWR028
+U 1 1 5703ABD0
+P 4800 2800
+F 0 "#PWR028" H 4800 2650 50  0001 C CNN
+F 1 "+5V" H 4800 2940 50  0000 C CNN
+F 2 "" H 4800 2800 50  0000 C CNN
+F 3 "" H 4800 2800 50  0000 C CNN
+	1    4800 2800
+	0    1    1    0
+$EndComp
+Wire Wire Line
+	4400 2800 4500 2800
+Wire Wire Line
+	4400 2400 4500 2400
+Wire Wire Line
+	4700 2550 4800 2550
+Wire Wire Line
+	4800 2550 4800 2400
+Wire Wire Line
+	4400 2400 4400 2250
+Text GLabel 6750 1950 3    60   Input ~ 0
+FLOW_INPUT
+Text GLabel 4650 4100 3    60   Input ~ 0
+FLOW_INPUT
 $EndSCHEMATC
