File: pcb/_autosave-RPi_Hat.kicad_pcb (KiCad board)
At the start: 2 copper layers, 65 x 56.5 mm, 43 parts, among them J1 RPi_GPIO, P1 Flow Meter, P2 Extra, P3 1 Wire, P4 Display, P5 Laser Controller Input, P6 Chiller/Air/Exhaust, Q1 BSS138, Q2 BSS138, Q4 BSS138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

Commit message: Update the schematic
Parts:
- moved JP2 0.64 mm to (132.1, 100.3)
Routing:
- net +5V: track 124.7 -> 124.0 mm
- net VSS: track 20.9 -> 20.3 mm
- net +24V: track 27.6 -> 27.0 mm
