File: pcb/_saved_RPi_Hat.sch (KiCad schematic (older format))
At the start: 39 parts, among them J1 RPi_GPIO, P1 Flow Meter, P2 Extra, P3 1 Wire, P4 Display, P5 Laser Controller Input, P6 Chiller/Air/Exhaust, Q1 BSS138, Q2 BSS138, Q4 BSS138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

Commit message: Update the schematic
Parts:
- JP2: footprint (none) -> Connect:PINHEAD1-3
Changed lines of the file:
@@
 F 0 "JP2" H 10000 3900 50  0000 L CNN
 F 1 "Relay Voltage Selector" H 9950 4100 50  0000 C BNN
-F 2 "" H 9950 4000 50  0000 C CNN
+F 2 "Connect:PINHEAD1-3" H 9950 4000 50  0001 C CNN
 F 3 "" H 9950 4000 50  0000 C CNN
 	1    9950 4000
